File: kicad/simple-battery-manager-v1/simple-battery-manager-v1.kicad_pcb (KiCad board)
At the start: 2 copper layers, 0 parts

Commit message: Initial layout of components. Pcb 25x25mm
Parts:
- added C1: 100nF, Capacitor_SMD:C_0805_2012Metric_Pad1.18x1.45mm_HandSolder, F.Cu at (157.5, 137.7)
- added C2: 100nF, Capacitor_SMD:C_0805_2012Metric_Pad1.18x1.45mm_HandSolder, F.Cu at (157.5, 126.7)
- added D1: SS14, Diode_SMD:D_SMA, F.Cu at (156.0, 121.2)
- added J1: BATT, Connector_PinHeader_2.54mm:PinHeader_1x02_P2.54mm_Vertical, F.Cu at (147.0, 142.2)
- added J2: DC-INPUT, Connector_PinHeader_2.54mm:PinHeader_1x02_P2.54mm_Vertical, F.Cu at (156.0, 142.2)
- added J3: OUTPUT, Connector_PinHeader_2.54mm:PinHeader_1x02_P2.54mm_Vertical, F.Cu at (163.2, 123.0)
- added J4: VBAT-CTRL, Connector_PinHeader_2.54mm:PinHeader_1x03_P2.54mm_Vertical, F.Cu at (163.0, 132.9)
- added JP1: JP-BATT, Connector_PinHeader_2.54mm:PinHeader_1x02_P2.54mm_Vertical, F.Cu at (142.0, 135.5)
- added JP2: SolderJumper_2_Open, Jumper:SolderJumper-2_P1.3mm_Open_TrianglePad1.0x1.5mm, F.Cu at (142.0, 129.2)
- added JP3: SolderJumper_2_Open, Jumper:SolderJumper-2_P1.3mm_Open_TrianglePad1.0x1.5mm, F.Cu at (142.0, 123.0)
- added Q1: Si2301DS, Package_TO_SOT_SMD:SOT-23_Handsoldering, F.Cu at (148.8, 136.0)
- added Q2: Si2301DS, Package_TO_SOT_SMD:SOT-23_Handsoldering, F.Cu at (148.5, 126.2)
- added R1: 100K, Resistor_SMD:R_0805_2012Metric_Pad1.20x1.40mm_HandSolder, F.Cu at (153.8, 137.7)
- added R2: 10K, Resistor_SMD:R_0805_2012Metric_Pad1.20x1.40mm_HandSolder, F.Cu at (153.8, 132.2)
- added R3: 10K, Resistor_SMD:R_0805_2012Metric_Pad1.20x1.40mm_HandSolder, F.Cu at (157.5, 132.2)
- added R4: 100K, Resistor_SMD:R_0805_2012Metric_Pad1.20x1.40mm_HandSolder, F.Cu at (153.8, 126.7)
Other:
- board outline added: 25 x 25 mm

Commit message: Layout and routing
Parts:
- C1, C2: footprint Capacitor_SMD:C_0805_2012Metric_Pad1.18x1.45mm_HandSolder -> Capacitor_SMD:C_0603_1608Metric_Pad1.08x0.95mm_HandSolder
- R1, R2, R3, R4: footprint Resistor_SMD:R_0805_2012Metric_Pad1.20x1.40mm_HandSolder -> Resistor_SMD:R_0603_1608Metric_Pad0.98x0.95mm_HandSolder
- moved J3 17.8 mm to (145.5, 123.0), turned to 90 degrees
- moved J4 13.8 mm to (153.4, 123.0), turned to 90 degrees
- moved D1 7.57 mm to (157.2, 128.7), turned to 180 degrees
- moved JP3 7.00 mm to (143.8, 129.8), turned to 90 degrees
- moved C2 6.56 mm to (159.5, 133.0), turned to 0 degrees
- moved R4 6.39 mm to (155.1, 133.0), turned to 0 degrees
- moved JP2 5.24 mm to (147.2, 129.8), turned to 90 degrees
- moved R3 4.42 mm to (159.4, 136.2), turned to 0 degrees
- moved Q2 4.19 mm to (150.8, 129.8)
- moved R2 4.16 mm to (154.9, 136.2), turned to 180 degrees
- moved C1 2.50 mm to (159.5, 139.2), turned to 180 degrees
- moved Q1 2.30 mm to (150.8, 137.0)
- moved JP1 2.17 mm to (143.8, 134.2)
- moved R1 1.91 mm to (154.9, 139.2), turned to 0 degrees
- moved J1 1.70 mm to (145.5, 143.0)
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Routing:
- net VCC: track 0.00 -> 32.3 mm, vias 0 -> 2
- net +BATT: track 0.00 -> 27.0 mm
- net /VBAT_READ_ENABLE: track 0.00 -> 22.1 mm, vias 0 -> 1
- net +5V: track 0.00 -> 21.9 mm, vias 0 -> 1
- net /VBAT_READ_OUTPUT: track 0.00 -> 19.0 mm, vias 0 -> 1
- net Net-(JP2-A): track 0.00 -> 10.9 mm
- net GND: track 0.00 -> 7.82 mm, vias 0 -> 9
- net Net-(J1-Pin_1): track 0.00 -> 6.98 mm
- added copper zone on B.Cu, net GND
- added copper zone on F.Cu, net GND
Other:
- board size 25 x 25 mm -> 20 x 20 mm
- board text added: "5V"
- board text added: "BATT"
- board text added: "GND"
- board text added: "Rev 1.0 04/24"
- board text added: "Simple Batt Mangager"
- board text added: "VBAT_EN"
- board text added: "VBAT_OUT"
- board text added: "VCC"
- board text added: "todo: confirm pin spacing for breadboard"

Commit message: pcb finished
Other:
- board text removed: "todo: confirm pin spacing for breadboard"
Changed lines of the file:
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@@
 		(rev "1.0")
 		(company "Gabriel Vega Engineering")
-		(comment 1 "Under Development")
+		(comment 1 "Finished")
 		(comment 2 "Gabriel Vega")
 		(comment 4 "1/1")
@@
 		)
 		(property "Value" "SolderJumper_2_Open"
-			(at 0 1.9 270)
+			(at 0 1.9 -90)
 			(layer "F.Fab")
 			(effects
@@
 		)
 		(property "Value" "10K"
-			(at 0 1.43 360)
+			(at 0 1.43 0)
 			(layer "F.Fab")
 			(effects
@@
 		)
 		(fp_text user "${REFERENCE}"
-			(at 0 0 360)
+			(at 0 0 0)
 			(layer "F.Fab")
 			(effects
@@
 		)
 		(property "Value" "SolderJumper_2_Open"
-			(at 0 1.9 270)
+			(at 0 1.9 -90)
 			(layer "F.Fab")
 			(effects
@@
 		)
 	)
-	(gr_text "todo:\n\nconfirm pin spacing for breadboard"
-		(at 173 138 0)
-		(layer "F.SilkS")
-		(effects
-			(font
-				(size 1 1)
-				(thickness 0.1)
-			)
-			(justify left bottom)
-		)
-	)
